File: AcousticDetection_HW/AcousticDetection_HW.kicad_pcb (KiCad board)
At the start: 2 copper layers, 203.9 x 67 mm, 22 parts, among them J1 USB_C_Receptacle_USB2.0, SW1 RST, U1 ESP32-WROOM-32, U2 LDL1117S33R_SOT223

Commit message: working on pcb layout
Parts:
- removed C11: 100nF, Capacitor_SMD:C_0805_2012Metric_Pad1.18x1.45mm_HandSolder
- added D1: POWER LED, LED_SMD:LED_0805_2012Metric_Pad1.15x1.40mm_HandSolder, B.Cu at (72.6, 73.7)
- added D2: INFO LED, LED_SMD:LED_0805_2012Metric_Pad1.15x1.40mm_HandSolder, B.Cu at (71.6, 84.3)
- added J10: PWR_R, AcousticDetection_extras:PowerConnector, B.Cu at (268.0, 63.0)
- added J11: DATA_R, AcousticDetection_extras:DataConnector, F.Cu at (54.4, 62.4)
- added J12: DATA_R, AcousticDetection_extras:DataConnector, F.Cu at (268.0, 63.0)
- added J2: BOOT OPTION, Connector_PinHeader_2.54mm:PinHeader_1x02_P2.54mm_Vertical, F.Cu at (130.3, 92.5)
- added J3: UART, Connector_PinHeader_2.54mm:PinHeader_1x04_P2.54mm_Vertical, F.Cu at (90.4, 76.7)
- added J4: JTAG, Connector_PinHeader_2.54mm:PinHeader_1x04_P2.54mm_Vertical, F.Cu at (68.6, 91.9)
- added J5: PWR_L, AcousticDetection_extras:PowerConnector, B.Cu at (90.4, 62.4)
- added J6: PWR_L, AcousticDetection_extras:PowerConnector, B.Cu at (99.0, 63.0)
- added J7: DATA_L, AcousticDetection_extras:DataConnector, F.Cu at (90.4, 62.4)
- added J8: DATA_L, AcousticDetection_extras:DataConnector, F.Cu at (99.0, 63.0)
- added J9: PWR_R, AcousticDetection_extras:PowerConnector, B.Cu at (54.4, 62.4)
- added R1: 5k1, Capacitor_SMD:C_0805_2012Metric_Pad1.18x1.45mm_HandSolder, F.Cu at (80.8, 95.0)
- added R2: 5k1, Capacitor_SMD:C_0805_2012Metric_Pad1.18x1.45mm_HandSolder, F.Cu at (80.8, 97.0)
- added R3: R, Capacitor_SMD:C_0805_2012Metric_Pad1.18x1.45mm_HandSolder, F.Cu at (70.1, 97.5)
- added R4: R, Capacitor_SMD:C_0805_2012Metric_Pad1.18x1.45mm_HandSolder, F.Cu at (73.7, 97.6)
- added SW2: BOOT, Button_Switch_SMD:SW_Tactile_SPST_NO_Straight_CK_PTS636Sx25SMTRLFS, F.Cu at (87.9, 87.4)
- C10, C7, C8, C9: footprint Capacitor_SMD:C_0603_1608Metric_Pad1.08x0.95mm_HandSolder -> Capacitor_SMD:C_0805_2012Metric_Pad1.18x1.45mm_HandSolder
- C2: footprint Capacitor_SMD:C_0805_2012Metric_Pad1.18x1.45mm_HandSolder -> Capacitor_SMD:C_1206_3216Metric_Pad1.33x1.80mm_HandSolder
- C4: footprint Capacitor_SMD:CP_Elec_5x3 -> Capacitor_SMD:C_1206_3216Metric_Pad1.33x1.80mm_HandSolder
- C5: value 100uF -> 10uF; footprint Capacitor_SMD:CP_Elec_6.3x7.7 -> Capacitor_SMD:C_1206_3216Metric_Pad1.33x1.80mm_HandSolder
- R6, R7, R8, R9: footprint Resistor_SMD:R_0603_1608Metric_Pad0.98x0.95mm_HandSolder -> Resistor_SMD:R_0805_2012Metric_Pad1.20x1.40mm_HandSolder
- SW1: value RST -> EN
- moved C3 59.7 mm to (61.0, 71.6), turned to -90 degrees
- moved C2 59.0 mm to (57.4, 72.1), turned to -90 degrees
- moved C1 51.0 mm to (61.0, 76.2), turned to 90 degrees
- moved C5 50.4 mm to (63.0, 94.0)
- moved R7 49.8 mm to (83.8, 78.7), turned to 90 degrees
- moved R5 46.9 mm to (56.9, 76.2)
- moved R6 43.5 mm to (84.3, 81.8)
- moved C4 42.9 mm to (64.5, 101.6)
- moved U2 40.8 mm to (57.9, 99.6)
- moved C6 38.5 mm to (54.9, 80.3), turned to 90 degrees
- moved SW1 25.2 mm to (56.4, 87.4)
- moved J1 23.0 mm to (88.0, 98.6), turned to 90 degrees
- moved U1 20.0 mm to (72.4, 79.4)
Connections:
- C10 pad 1: GND -> /GND_R
- C10 pad 2: +3.3V -> /3V3_R
- C6 pad 1: +3.3V -> GND
- C6 pad 2: GND -> EN
- C7 pad 1: GND -> /GND_L
- C7 pad 2: +3.3V -> Net-(J6-3V3)
- C8 pad 1: GND -> /GND_R
- C8 pad 2: +3.3V -> /3V3_R
- C9 pad 1: GND -> /GND_L
- C9 pad 2: +3.3V -> Net-(J6-3V3)
- MK1-left1 pad 1: WS -> /WS_L
- MK1-left1 pad 2: GND -> /GND_L
- MK1-left1 pad 3: GND -> /GND_L
- MK1-left1 pad 4: BCLK -> /BCLK_L
- MK1-left1 pad 5: +3.3V -> Net-(J6-3V3)
- MK2-right1 pad 1: WS -> /WS_R
- MK2-right1 pad 2: +3.3V -> /3V3_R
- MK2-right1 pad 3: GND -> /GND_R
- MK2-right1 pad 4: BCLK -> /BCLK_R
- MK2-right1 pad 5: +3.3V -> /3V3_R
- R8 pad 2: MIC_DATA -> /MIC_DATA_L
- R9 pad 2: MIC_DATA -> /MIC_DATA_R
- U1 pad 24: unconnected-(U1-IO2-Pad24) -> INFO_LED
- U1 pad 34: Net-(J3-Pin_3) -> /RXD
- U1 pad 35: Net-(J3-Pin_2) -> /TXD
Routing:
- net GND: track 17.0 -> 0.00 mm
- net BCLK: track 14.3 -> 0.00 mm
- net WS: track 13.8 -> 0.00 mm
- net +3.3V: track 12.8 -> 0.00 mm, vias 2 -> 0
- net /GND_L: track 0.00 -> 10.6 mm
- net /3V3_R: track 0.00 -> 9.17 mm, vias 0 -> 2
- net /BCLK_R: track 0.00 -> 7.69 mm
- net /WS_R: track 0.00 -> 7.05 mm
- net /WS_L: track 0.00 -> 6.78 mm
- net /BCLK_L: track 0.00 -> 6.57 mm
- net /GND_R: track 0.00 -> 6.46 mm
- net MIC_DATA: track 4.74 -> 0.00 mm
- net Net-(J6-3V3): track 0.00 -> 3.64 mm
- net /MIC_DATA_R: track 0.00 -> 2.50 mm
- net /MIC_DATA_L: track 0.00 -> 2.23 mm
Other:
- board size 203.9 x 67 mm -> 217.6 x 45 mm
- board text added: "3V3"
- board text added: "GND"
- board text added: "RXD"
- board text added: "TXD"

Commit message: finishing pcb
Parts:
- removed J2: BOOT OPTION, Connector_PinHeader_2.54mm:PinHeader_1x02_P2.54mm_Vertical
- added G***: LOGO, LOGO, B.Cu at (177.3, 63.0)
- added G***: LOGO, LOGO, B.Cu at (34.8, 98.8)
- added G***: LOGO, LOGO, B.Cu at (189.7, 63.0)
- C10, C7, C8, C9: footprint Capacitor_SMD:C_0805_2012Metric_Pad1.18x1.45mm_HandSolder -> Capacitor_SMD:C_0603_1608Metric_Pad1.08x0.95mm_HandSolder
- C3: value 100n -> 100nF
- D1: value POWER LED -> POWER; footprint LED_SMD:LED_0805_2012Metric_Pad1.15x1.40mm_HandSolder -> LED_SMD:LED_1206_3216Metric_Pad1.42x1.75mm_HandSolder
- D2: value INFO LED -> INFO; footprint LED_SMD:LED_0805_2012Metric_Pad1.15x1.40mm_HandSolder -> LED_SMD:LED_1206_3216Metric_Pad1.42x1.75mm_HandSolder
- R1, R2: footprint Capacitor_SMD:C_0805_2012Metric_Pad1.18x1.45mm_HandSolder -> Resistor_SMD:R_0805_2012Metric_Pad1.20x1.40mm_HandSolder
- R3, R4: value R -> 1k; footprint Capacitor_SMD:C_0805_2012Metric_Pad1.18x1.45mm_HandSolder -> Resistor_SMD:R_0805_2012Metric_Pad1.20x1.40mm_HandSolder
- R8, R9: footprint Resistor_SMD:R_0805_2012Metric_Pad1.20x1.40mm_HandSolder -> Resistor_SMD:R_0603_1608Metric_Pad0.98x0.95mm_HandSolder
- moved J3 32.5 mm to (57.9, 77.2)
- moved C1 31.5 mm to (29.5, 77.2)
- moved J5 31.5 mm to (58.9, 63.0)
- moved J7 31.5 mm to (58.9, 63.0)
- moved J1 31.3 mm to (56.7, 98.3)
- moved R1 31.1 mm to (49.8, 97.0)
- moved R2 31.1 mm to (49.8, 99.1), turned to 180 degrees
- moved SW2 31.0 mm to (56.9, 87.9)
- moved C5 29.9 mm to (33.1, 94.0), turned to 180 degrees
- moved D1 29.8 mm to (42.9, 73.7)
- moved J4 29.5 mm to (39.1, 92.5)
- moved R5 29.5 mm to (27.4, 77.2), turned to 90 degrees
- moved R6 29.5 mm to (54.8, 82.1)
- moved C2 29.5 mm to (27.9, 72.7)
- moved C3 29.5 mm to (31.5, 72.2)
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Connections:
- net Net-(J6-3V3) renamed /3V3_L
Routing:
- net GND: track 0.00 -> 263.2 mm, vias 0 -> 5
- net +3.3V: track 0.00 -> 123.2 mm, vias 0 -> 1
- net /3V3_L: track 3.64 -> 79.8 mm, vias 0 -> 1
- net /3V3_R: track 9.17 -> 85.3 mm, vias 2 -> 3
- net /GND_R: track 6.46 -> 81.7 mm, vias 0 -> 1
- net /GND_L: track 10.6 -> 84.7 mm, vias 0 -> 1
- net /BCLK_L: track 6.57 -> 80.1 mm
- net /MIC_DATA_L: track 2.23 -> 75.7 mm
- net /MIC_DATA_R: track 2.50 -> 75.6 mm
- net /BCLK_R: track 7.69 -> 80.4 mm
- net /WS_R: track 7.05 -> 79.3 mm
- net /WS_L: track 6.78 -> 78.8 mm
- net BCLK: track 0.00 -> 59.9 mm
- net WS: track 0.00 -> 56.0 mm, vias 0 -> 2
- net MIC_DATA: track 0.00 -> 51.3 mm, vias 0 -> 4
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- added copper zone on B.Cu, net /GND_L
- added copper zone on F.Cu, net /GND_L
- added copper zone on B.Cu, net /GND_R
- added copper zone on F.Cu, net /GND_R
- added copper zone on B.Cu, net GND
- added copper zone on F.Cu, net GND
Other:
- board size 217.6 x 45 mm -> 247.1 x 104.3 mm
- board text added: "Acoustic Detection v1.0 Matěj Trnka 4/2023"
- board text added: "Acoustic Detection v1.0, Matěj Trnka, 4/2023"
- board text added: "České vysoké učení technické v Praze"

Commit message: cleanup
Parts:
- moved R9 148.0 mm to (48.1, 81.4)
- moved C10 148.0 mm to (48.7, 83.9)
- moved C8 148.0 mm to (47.1, 83.9)
- moved G*** 148.0 mm to (43.1, 82.9)
- moved J10 148.0 mm to (123.4, 82.9)
- moved J12 148.0 mm to (123.4, 82.9)
- moved MK2-right1 148.0 mm to (43.4, 82.9)
- moved C1 103.5 mm to (131.1, 97.0)
- moved C3 103.5 mm to (133.1, 92.0)
- moved D1 103.5 mm to (144.5, 93.4)
- moved D2 103.5 mm to (144.5, 102.3)
- moved G*** 103.5 mm to (136.4, 118.6)
- moved J4 103.5 mm to (140.7, 112.3)
- moved R1 103.5 mm to (151.4, 116.8)
- moved R2 103.5 mm to (151.4, 118.8)
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Other:
- board size 247.1 x 104.3 mm -> 208 x 44 mm
- board text removed: "Acoustic Detection v1.0 Matěj Trnka 4/2023"

Commit message: small changes
Other:
- board text added: "Acoustic Detection v1.0, Matěj Trnka 4/2023"
- board text removed: "Acoustic Detection v1.0, Matěj Trnka, 4/2023"
Changed lines of the file:
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@@
         (effects (font (size 1 1) (thickness 0.15)) (justify mirror))
     )
-    (fp_text value "PWR_R" (at -0.254 -4.572 unlocked) (layer "B.Fab")
+    (fp_text value "PWR_R" (at 8.544 0.131 unlocked) (layer "B.Fab")
         (effects (font (size 1 1) (thickness 0.15)) (justify mirror))
     )
@@
         (effects (font (size 1 1) (thickness 0.15)) (justify left bottom mirror))
     )
-    (fp_text user "${REFERENCE}" (at 0 -6.35 unlocked) (layer "B.Fab")
+    (fp_text user "${REFERENCE}" (at 9.052 1.147 unlocked) (layer "B.Fab")
         (effects (font (size 1 1) (thickness 0.15)) (justify mirror))
     )
@@
         (effects (font (size 1 1) (thickness 0.15)) (justify mirror))
     )
-    (fp_text value "PWR_R" (at 0 4.504 unlocked) (layer "B.Fab")
+    (fp_text value "PWR_R" (at -4.072 1.964 unlocked) (layer "B.Fab")
         (effects (font (size 1 1) (thickness 0.15)) (justify mirror))
     )
@@
         (effects (font (size 1 1) (thickness 0.15)) (justify left bottom mirror))
     )
-    (fp_text user "${REFERENCE}" (at 3.556 -0.068 unlocked) (layer "B.Fab")
+    (fp_text user "${REFERENCE}" (at -5.596 0.948 unlocked) (layer "B.Fab")
         (effects (font (size 1 1) (thickness 0.15)) (justify mirror))
     )
@@
         (effects (font (size 1 1) (thickness 0.15)) (justify mirror))
     )
-    (fp_text value "PWR_L" (at -0.068 3.996 unlocked) (layer "B.Fab")
+    (fp_text value "PWR_L" (at 4.052 1.964 unlocked) (layer "B.Fab")
         (effects (font (size 1 1) (thickness 0.15)) (justify mirror))
     )
@@
         (effects (font (size 1 1) (thickness 0.15)) (justify left bottom mirror))
     )
-    (fp_text user "${REFERENCE}" (at -3.116 -0.068 unlocked) (layer "B.Fab")
+    (fp_text user "${REFERENCE}" (at 5.068 0.44 unlocked) (layer "B.Fab")
         (effects (font (size 1 1) (thickness 0.15)) (justify mirror))
     )
@@
         (effects (font (size 1 1) (thickness 0.15)) (justify mirror))
     )
-    (fp_text value "PWR_L" (at -0.254 -4.572 unlocked) (layer "B.Fab")
+    (fp_text value "PWR_L" (at -7.92 -1.016 unlocked) (layer "B.Fab")
         (effects (font (size 1 1) (thickness 0.15)) (justify mirror))
     )
@@
         (effects (font (size 1 1) (thickness 0.15)) (justify left bottom mirror))
     )
-    (fp_text user "${REFERENCE}" (at 0 -6.35 unlocked) (layer "B.Fab")
+    (fp_text user "${REFERENCE}" (at -8.936 0.508 unlocked) (layer "B.Fab")
         (effects (font (size 1 1) (thickness 0.15)) (justify mirror))
     )
@@
     (effects (font (size 1.2 1.2) (thickness 0.18)) (justify left bottom))
   )
-  (gr_text "Acoustic Detection v1.0, Matěj Trnka, 4/2023" (at 61.976 83.82) (layer "F.SilkS")
+  (gr_text "Acoustic Detection v1.0, Matěj Trnka 4/2023" (at 61.976 83.82) (layer "F.SilkS")
     (effects (font (size 1.2 1.2) (thickness 0.18)) (justify left bottom))
   )

Commit message: parts labels reposition
Parts:
- moved G*** 112.5 mm to (146.3, 135.6), turned to 90 degrees
- moved MK1-left1 112.1 mm to (146.3, 135.3), turned to 0 degrees
- moved C7 107.4 mm to (145.3, 131.6), turned to 0 degrees
- moved C9 105.4 mm to (145.3, 130.0), turned to 0 degrees
- moved R8 105.1 mm to (147.8, 130.7), turned to 90 degrees
- moved G*** 77.0 mm to (99.3, 135.6), turned to -90 degrees
- moved MK2-right1 76.7 mm to (99.3, 135.3), turned to 0 degrees
- moved C8 71.4 mm to (100.3, 131.6), turned to 180 degrees
- moved R9 70.0 mm to (97.8, 130.6), turned to 90 degrees
- moved C10 69.2 mm to (100.3, 130.0), turned to 180 degrees
- moved J10 36.6 mm to (99.3, 55.3), turned to -90 degrees
- moved J12 36.6 mm to (99.3, 55.3), turned to -90 degrees
- moved C1 34.2 mm to (109.4, 70.6)
- moved R1 34.2 mm to (129.7, 90.4)
- moved R2 34.2 mm to (129.7, 92.5)
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Other:
- board size 208 x 44 mm -> 53 x 85 mm

Commit message: pcb fabrication
Parts:
- moved C1 30.0 mm to (139.3, 71.6)
- moved C2 30.0 mm to (137.8, 67.1)
- moved C5 30.0 mm to (142.9, 88.4)
- moved C6 30.0 mm to (141.4, 71.6)
- moved C7 30.0 mm to (175.3, 132.6)
- moved C9 30.0 mm to (175.3, 131.1)
- moved D1 30.0 mm to (152.7, 68.1)
- moved D2 30.0 mm to (152.7, 77.0)
- moved G*** 30.0 mm to (176.3, 136.7)
- moved G*** 30.0 mm to (144.7, 93.2)
- moved J1 30.0 mm to (166.6, 92.7)
- moved J11 30.0 mm to (136.8, 57.4)
- moved J3 30.0 mm to (167.8, 71.6)
- moved J5 30.0 mm to (168.8, 57.4)
- moved J6 30.0 mm to (176.3, 56.4)
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
Commit message: the resistor values of pcb leds were changed to 220R
Parts:
- R3, R4: value 1k -> 220R
Changed lines of the file:
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@@
         (effects (font (size 1 1) (thickness 0.15)))
     )
-    (fp_text value "1k" (at 0 1.65 90) (layer "F.Fab")
+    (fp_text value "220R" (at 0 1.65 90) (layer "F.Fab")
         (effects (font (size 1 1) (thickness 0.15)))
     )
@@
         (effects (font (size 1 1) (thickness 0.15)))
     )
-    (fp_text value "1k" (at 0 1.65 90) (layer "F.Fab")
-        (effects (font (size 1 1) (thickness 0.15)))
-    )
+    (fp_text value "220R" (at 0 1.65 90) (layer "F.Fab")
+        (effects (font (size 1 1) (thickness 0.15)))
+    )
